File: schematic/Yet-Another-LED-Cube.brd (EAGLE design)
At the start: 160 x 100 mm, 7 parts, among them IC1 7805T, J1 DCJ0202

Commit message: added a bunch of parts
Parts:
- added IC2: MEGA48/88/168-PU, avr-6:DIL28-3
- added IC3, IC4: 74HC164N, 74xx-eu:DIL14
- added Q1, Q10, Q11, Q12, Q13, Q14, Q15, Q16, Q2, Q3, Q4, Q5, Q6, Q7, Q8, Q9: 2N2907, transistor-pnp:TO18
- added R1, R11, R13, R15, R17, R19, R21, R23, R25, R27, R29, R3, R31, R5, R7, R9: 1K, resistor:0204V
- added R10, R12, R14, R16, R18, R2, R20, R22, R24, R26, R28, R30, R32, R33, R4, R6, R8: 10K, resistor:0204V
- added U1: TLC5940-RHB, SparkFun:QFN-32
Connections:
- new net AGND: IC2.22
- new net N$11: IC3.12, R5.1
- new net N$12: IC3.11, R3.1
- new net N$13: IC3.10, R1.1
- new net N$14: IC3.3, R9.1
- new net N$15: IC3.4, R11.1
- new net N$16: IC3.5, R13.1
- new net N$17: IC3.6, R15.1
- new net N$19: Q9.2, R17.2, R18.1
- new net N$2: Q1.2, R1.2, R2.1
- new net N$20: Q10.2, R19.2, R20.1
- new net N$21: Q11.2, R21.2, R22.1
- new net N$22: Q12.2, R23.2, R24.1
- new net N$23: Q13.2, R25.2, R26.1
- new net N$24: Q14.2, R27.2, R28.1
- new net N$25: Q15.2, R29.2, R30.1
- new net N$26: Q16.2, R31.2, R32.1
- new net N$27: IC4.13, R23.1
- new net N$28: IC4.12, R21.1
- new net N$29: IC4.11, R19.1
- new net N$3: Q2.2, R3.2, R4.1
- new net N$30: IC4.10, R17.1
- new net N$31: IC4.3, R25.1
- new net N$32: IC4.4, R27.1
- new net N$33: IC4.5, R29.1
- new net N$34: IC4.6, R31.1
- new net N$35: Q1.1, Q10.1, Q11.1, Q12.1, Q13.1, Q14.1, Q15.1, Q16.1, Q2.1, Q3.1, Q4.1, Q5.1, Q6.1, Q7.1, Q8.1, Q9.1, R10.2, R12.2, R14.2, R16.2, R18.2, R2.2, R20.2, R22.2, R24.2, R26.2, R28.2, R30.2, R32.2, R4.2, R6.2, R8.2
- new net N$36: IC3.9, IC4.9, R33.1
- new net N$37: IC3.1, IC3.2
- new net N$39: IC3.8, IC4.8
- new net N$4: Q3.2, R5.2, R6.1
- new net N$40: IC3.13, IC4.1, IC4.2, R7.1
- new net N$5: Q4.2, R7.2, R8.1
- new net N$6: Q5.2, R10.1, R9.2
- new net N$7: Q6.2, R11.2, R12.1
- new net N$8: Q7.2, R13.2, R14.1
- new net N$9: Q8.2, R15.2, R16.1
- new net VCC: IC2.7, IC3.14, IC4.14
- net +5V: now also R33.2
- net GND: now also IC1.2, IC2.8, IC3.7, IC4.7

Commit message: Add RGB LED parts; connect IC's
Parts:
- added C5: 10nF, rcl:C025-024X044
- added C6, C7: 100nF, rcl:C025-024X044
- added C8, C9: 18pF, rcl:C025-024X044
- added LED1, LED10, LED11, LED12, LED13, LED14, LED15, LED16, LED17, LED18, LED19, LED2, LED20, LED21, LED22, LED23, LED24, LED25, LED26, LED27, LED28, LED29, LED3, LED30, LED31, LED32, LED33, LED34, LED35, LED36, LED37, LED38, LED39, LED4, LED40, LED41, LED42, LED43, LED44, LED45, LED46, LED47, LED48, LED49, LED5, LED50, LED51, LED52, LED53, LED54, LED55, LED56, LED57, LED58, LED59, LED6, LED60, LED61, LED62, LED63, LED64, LED7, LED8, LED9: RGBLED_CAA, adafruit:LED5MMRGB2
- added Q17: 20MHz, crystal:HC49/S
- added R34: 330, resistor:0204V
- added R35: 3K3, resistor:0204V
- added R36, R37: 10K, resistor:0204V
- moved Q9 328.0 mm to (-2.54, -468.6)
- moved Q10 323.9 mm to (-38.1, -476.2)
- moved Q11 323.9 mm to (-24.1, -476.2)
- moved R20 318.8 mm to (-39.4, -488.9)
- moved R21 318.8 mm to (-34.3, -488.9)
- moved Q12 318.7 mm to (-10.2, -476.2)
- moved Q13 318.7 mm to (3.81, -476.2)
- moved Q14 317.5 mm to (-38.1, -482.6)
- moved Q15 317.5 mm to (-24.1, -482.6)
- moved Q16 312.4 mm to (-10.2, -482.6)
- moved R17 312.4 mm to (2.54, -482.6)
- moved R18 312.4 mm to (7.62, -482.6)
- moved R19 312.4 mm to (12.7, -482.6)
- moved R32 311.5 mm to (-39.4, -495.3)
- moved R22 311.3 mm to (-29.2, -488.9)
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Connections:
- removed net AGND: IC2.22
- removed net N$40 (its old number): IC3.13, IC4.1, IC4.2, R7.1
- new net N$10: LED1.P$1, LED13.P$1, LED17.P$1, LED21.P$1, LED25.P$1, LED29.P$1, LED33.P$1, LED34.P$1, LED41.P$1, LED45.P$1, LED49.P$1, LED5.P$1, LED53.P$1, LED57.P$1, LED61.P$1, LED9.P$1, U1.4
- new net N$124: LED29.P$2, LED30.P$2, LED31.P$2, LED32.P$2, Q4.3
- new net N$125: LED25.P$2, LED26.P$2, LED27.P$2, LED28.P$2, Q3.3
- new net N$126: LED21.P$2, LED22.P$2, LED23.P$2, LED24.P$2, Q2.3
- new net N$127: LED17.P$2, LED18.P$2, LED19.P$2, LED20.P$2, Q1.3
- new net N$128: LED13.P$2, LED14.P$2, LED15.P$2, LED16.P$2, Q8.3
- new net N$129: LED10.P$2, LED11.P$2, LED12.P$2, LED9.P$2, Q7.3
- new net N$18: LED1.P$3, LED13.P$3, LED17.P$3, LED21.P$3, LED25.P$3, LED29.P$3, LED33.P$3, LED34.P$3, LED41.P$3, LED45.P$3, LED49.P$3, LED5.P$3, LED53.P$3, LED57.P$3, LED61.P$3, LED9.P$3, U1.5
- new net N$34: IC2.19, U1.1
- new net N$35: LED1.P$2, LED2.P$2, LED3.P$2, LED4.P$2, Q5.3
- new net N$36: IC2.12, IC3.8, IC4.8
- new net N$38: LED1.P$4, LED13.P$4, LED17.P$4, LED21.P$4, LED25.P$4, LED29.P$4, LED33.P$4, LED34.P$4, LED41.P$4, LED45.P$4, LED49.P$4, LED5.P$4, LED53.P$4, LED57.P$4, LED61.P$4, LED9.P$4, U1.6
- new net N$41: LED5.P$2, LED6.P$2, LED7.P$2, LED8.P$2, Q6.3
- new net N$42: LED10.P$1, LED14.P$1, LED18.P$1, LED2.P$1, LED22.P$1, LED26.P$1, LED30.P$1, LED35.P$1, LED36.P$1, LED42.P$1, LED46.P$1, LED50.P$1, LED54.P$1, LED58.P$1, LED6.P$1, LED62.P$1, U1.7
- new net N$43: LED10.P$3, LED14.P$3, LED18.P$3, LED2.P$3, LED22.P$3, LED26.P$3, LED30.P$3, LED35.P$3, LED36.P$3, LED42.P$3, LED46.P$3, LED50.P$3, LED54.P$3, LED58.P$3, LED6.P$3, LED62.P$3, U1.8
- new net N$44: LED10.P$4, LED14.P$4, LED18.P$4, LED2.P$4, LED22.P$4, LED26.P$4, LED30.P$4, LED35.P$4, LED36.P$4, LED42.P$4, LED46.P$4, LED50.P$4, LED54.P$4, LED58.P$4, LED6.P$4, LED62.P$4, U1.9
- new net N$45: IC3.13, R7.1
- new net N$46: LED11.P$1, LED15.P$1, LED19.P$1, LED23.P$1, LED27.P$1, LED3.P$1, LED31.P$1, LED37.P$1, LED38.P$1, LED43.P$1, LED47.P$1, LED51.P$1, LED55.P$1, LED59.P$1, LED63.P$1, LED7.P$1, U1.10
- new net N$47: LED11.P$3, LED15.P$3, LED19.P$3, LED23.P$3, LED27.P$3, LED3.P$3, LED31.P$3, LED37.P$3, LED38.P$3, LED43.P$3, LED47.P$3, LED51.P$3, LED55.P$3, LED59.P$3, LED63.P$3, LED7.P$3, U1.11
- new net N$48: LED11.P$4, LED15.P$4, LED19.P$4, LED23.P$4, LED27.P$4, LED3.P$4, LED31.P$4, LED37.P$4, LED38.P$4, LED43.P$4, LED47.P$4, LED51.P$4, LED55.P$4, LED59.P$4, LED63.P$4, LED7.P$4, U1.14
- new net N$49: IC2.18, U1.23
- new net N$50: LED12.P$1, LED16.P$1, LED20.P$1, LED24.P$1, LED28.P$1, LED32.P$1, LED39.P$1, LED4.P$1, LED40.P$1, LED44.P$1, LED48.P$1, LED52.P$1, LED56.P$1, LED60.P$1, LED64.P$1, LED8.P$1, U1.15
- new net N$51: LED12.P$3, LED16.P$3, LED20.P$3, LED24.P$3, LED28.P$3, LED32.P$3, LED39.P$3, LED4.P$3, LED40.P$3, LED44.P$3, LED48.P$3, LED52.P$3, LED56.P$3, LED60.P$3, LED64.P$3, LED8.P$3, U1.16
- new net N$52: LED12.P$4, LED16.P$4, LED20.P$4, LED24.P$4, LED28.P$4, LED32.P$4, LED39.P$4, LED4.P$4, LED40.P$4, LED44.P$4, LED48.P$4, LED52.P$4, LED56.P$4, LED60.P$4, LED64.P$4, LED8.P$4, U1.17
- new net N$54: IC2.15, U1.32
- new net N$55: IC2.5, R35.2
- new net N$56: IC2.16, R36.1, U1.31
- new net N$57: IC2.14, U1.3
- new net N$58: R34.2, U1.26
- new net N$59: R35.1, U1.24
- new net N$60: R37.1, U1.25
- new net N$61: LED33.P$2, LED35.P$2, LED37.P$2, LED39.P$2, Q13.3
- new net N$62: LED34.P$2, LED36.P$2, LED38.P$2, LED40.P$2, Q14.3
- new net N$63: LED61.P$2, LED62.P$2, LED63.P$2, LED64.P$2, Q12.3
- new net N$64: LED57.P$2, LED58.P$2, LED59.P$2, LED60.P$2, Q11.3
- new net N$65: LED53.P$2, LED54.P$2, LED55.P$2, LED56.P$2, Q10.3
- new net N$66: LED49.P$2, LED50.P$2, LED51.P$2, LED52.P$2, Q9.3
- new net N$67: LED45.P$2, LED46.P$2, LED47.P$2, LED48.P$2, Q16.3
- new net N$68: LED41.P$2, LED42.P$2, LED43.P$2, LED44.P$2, Q15.3
- new net N$70: C6.1, IC2.21
- new net N$72: C8.2, IC2.9, Q17.2
- new net N$73: C9.2, IC2.10, Q17.1
- net +5V: now also C5.1, C7.1, IC2.20, IC2.7, R36.2, R37.2, U1.27
- net GND: now also C5.2, C6.2, C7.2, C8.1, C9.1, IC2.22, R34.1, U1.30
- net N$37: now also IC4.1, IC4.2
- net N$39: now also IC2.17, U1.2; no longer IC3.8, IC4.8
- net VCC: no longer IC2.7
